Commit message: mpc mhe working

File: quads/hummingbird/hummingbird.xacro (robot description, xacro)
@@ -34,5 +34,5 @@
   <xacro:property name="time_constant_up" value="0.0125" /> <!-- [s] -->
   <xacro:property name="time_constant_down" value="0.025" /> <!-- [s] -->
-  <xacro:property name="max_rot_velocity" value="1000" /> <!-- 838 [rad/s] -->
+  <xacro:property name="max_rot_velocity" value="838" /> <!-- 838 [rad/s] -->
   <xacro:property name="rotor_drag_coefficient" value="8.06428e-05" /> <!-- 8.06428e-05 -->
   <xacro:property name="rolling_moment_coefficient" value="0.000001" />
